File: fpga.kicad_sch (KiCad schematic)
At the start: 9 parts

Commit message: Added programmer for FPGA
Parts:
- added U4: FT2232HQ, Package_DFN_QFN:QFN-64-1EP_9x9mm_P0.5mm_EP4.35x4.35mm, symbol Interface_USB:FT2232HQ
Other:
- note removed: "3.2.2 FPGA reset using the POR module Using the POR module, in many cases no external components are required to ensure a safe reset of the GateMate FPGA. Figure 3.4 shows how to connect the reset pins in this case: • VDD_WA and VDD_CLK must be connected to 1.1 . . 2.7 V supply (might be different). • POR_EN has to be connected to VDD_WA or it can be left open due to the internal pullup resistor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"
- note removed: "The POR must be enabled with POR_EN signal: 0: Reset state depends only on the RST_N signal. 1: FPGA changes from reset to operation state when RST_N is 1 and POR indicates VDD and VDD_CLK voltages are stable."
- note removed: "The section you've provided describes the Power-On Reset (POR) feature of the GateMate™ FPGA. This is an important aspect of the FPGA's power-up sequence, ensuring that it starts up correctly under the right conditions. Here's a breakdown of what this means and how you would typically power on the FPGA: Reset Pin (RST_N): The FPGA has a reset pin labeled RST_N. This pin is active low, meaning it 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"
Changed lines of the file:
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@@
-		)
-	)
-	(text "The POR must be enabled with POR_EN signal:\n0: Reset state depends only on the RST_N signal.\n1: FPGA changes from reset to operation state when RST_N is 1 and POR indicates VDD\nand VDD_CLK voltages are stable."
-		(exclude_from_sim no)
-		(at 25.4 275.59 0)
-		(effects
-			(font
-				(size 1.27 1.27)
-			)
-			(justify left bottom)
-		)
-	)
-	(text "The section you've provided describes the Power-On Reset (POR) feature of the GateMate™ FPGA. This is an important aspect of the FPGA's power-up sequence, ensuring that it starts up correctly under the right conditions. Here's a breakdown of what this means and how you would typically power on the FPGA:\n\nReset Pin (RST_N): The FPGA has a reset pin labeled RST_N. This pin is active low, meaning it activates or triggers a reset when it is pulled to a low voltage level. The Schmitt-trigger characteristic refers to the input having hysteresis, making it less sensitive to noise on the reset signal. The internal pull-up resistor means the reset pin will be in a non-active (high) state when not externally driven low.\n\nPower-On Reset (POR) Module: The POR module is an internal feature of the FPGA that ensures the device starts up safely when power is applied. It monitors the core voltage (VDD) and the clock supply voltage (VDD_CLK).\n\nSafe Reset Generation: Once VDD and VDD_CLK are stable and within their specified ranges, the POR module generates a safe reset signal. This ensures that the FPGA starts in a known state.\nVoltage Drop Detection: The POR module can detect a drop in the VDD and VDD_CLK voltages, which might require a reset to maintain proper operation.\nAdjustable VDD_CLK Voltage Threshold: You can set a threshold for the VDD_CLK voltage, allowing flexibility depending on your specific power supply setup.\nNo Restrictions on Voltage Switch-On Order: You don't need to power on VDD and VDD_CLK in any particular order. The FPGA can handle either being powered first.\nTurning On the FPGA: To power on the FPGA:\n\nApply Power: Ensure that both the core voltage (VDD) and the clock supply voltage (VDD_CLK) are connected and meet the FPGA's voltage requirements.\nNo Need to Manually Reset: Thanks to the internal POR module, the FPGA will automatically reset itself once it detects that the VDD and VDD_CLK voltages are stable. You don't need to manually activate the RST_N pin unless you want to reset the FPGA during operation."
-		(exclude_from_sim no)
-		(at 128.27 142.24 0)
-		(effects
-			(font
-				(size 1.27 1.27)
-			)
-			(justify left bottom)
-		)
-	)
-	(text "3.2.2 FPGA reset using the POR module\nUsing the POR module, in many cases no external components are required to ensure a\nsafe reset of the GateMate FPGA. Figure 3.4 shows how to connect the reset pins in this\ncase:\n• VDD_WA and VDD_CLK must be connected to 1.1 . . 2.7 V supply (might be different).\n• POR_EN has to be connected to VDD_WA or it can be left open due to the internal pullup resistor.\n• Pin RST_N must be connected to VDD_CLK.\n• In normal operation, POR_ADJ should be left open. The optional voltage divider R3a\nand R3b is only used, if POR adjustment is required. This depends on the VDD_CLK\nlevel (see explanation below).\n\n\n-> This means the FPGA itself knows how to power on. We will start through a reset.\n"
-		(exclude_from_sim no)
-		(at 102.87 254 0)
-		(effects
-			(font
-				(size 1.27 1.27)
-			)
-			(justify left bottom)
 		)
 	)
@@
 					(unit 1)
 				)
+			)
+		)
+	)
+	(symbol
+		(lib_id "Interface_USB:FT2232HQ")
+		(at 369.57 85.09 0)
+		(unit 1)
+		(exclude_from_sim no)
+		(in_bom yes)
+		(on_board yes)
+		(dnp no)
+		(fields_autoplaced yes)
+		(property "Reference" "U4"
+			(at 384.4641 27.94 0)
+			(effects
+				(font
+					(size 1.27 1.27)
+				)
+				(justify left)
+			)
+		)
+		(property "Value" "FT2232HQ"
+			(at 384.4641 30.48 0)
+			(effects
+				(font
+					(size 1.27 1.27)
+				)
+				(justify left)
+			)
+		)
+		(property "Footprint" "Package_DFN_QFN:QFN-64-1EP_9x9mm_P0.5mm_EP4.35x4.35mm"
+			(at 369.57 85.09 0)
+			(effects
+				(font
+					(size 1.27 1.27)
+				)
+				(hide yes)
+			)
+		)
+		(property "Datasheet" "https://www.ftdichip.com/Support/Documents/DataSheets/ICs/DS_FT2232H.pdf"
+			(at 369.57 85.09 0)
+			(effects
+				(font
+					(size 1.27 1.27)
+				)
+				(hide yes)
+			)
+		)
+		(property "Description" "Hi Speed Double Channel USB UART/FIFO, QFN-64"
+			(at 369.57 85.09 0)
+			(effects
+				(font
+					(size 1.27 1.27)
+				)
+				(hide yes)
+			)
+		)
+		(pin "34"
+		)
+		(pin "17"
+		)
+		(pin "46"
+		)
+		(pin "33"
+		)
+		(pin "20"
+		)
+		(pin "43"
+		)
+		(pin "26"
+		)
+		(pin "18"
+		)
+		(pin "51"
+		)
+		(pin "54"
+		)
+		(pin "32"
+		)
+		(pin "58"
+		)
+		(pin "22"
+		)
+		(pin "23"
+		)
+		(pin "29"
+		)
+		(pin "44"
+		)
+		(pin "39"
+		)
+		(pin "41"
+		)
+		(pin "53"
+		)
+		(pin "37"
+		)
+		(pin "49"
+		)
+		(pin "47"
+		)
+		(pin "11"
+		)
+		(pin "35"
+		)
+		(pin "5"
+		)
+		(pin "56"
+		)
+		(pin "61"
+		)
+		(pin "25"
+		)
+		(pin "48"
+		)
+		(pin "14"
+		)
+		(pin "19"
+		)
+		(pin "40"
+		)
+		(pin "6"
+		)
+		(pin "62"
+		)
+		(pin "64"
+		)
+		(pin "52"
+		)
+		(pin "4"
+		)
+		(pin "42"
+		)
+		(pin "50"
+		)
+		(pin "3"
+		)
+		(pin "2"
+		)
+		(pin "24"
+		)
+		(pin "21"
+		)
+		(pin "12"
+		)
+		(pin "1"
+		)
+		(pin "27"
+		)
+		(pin "15"
+		)
+		(pin "38"
+		)
+		(pin "55"
+		)
+		(pin "57"
+		)
+		(pin "45"
+		)
+		(pin "59"
+		)
+		(pin "28"
+		)
+		(pin "10"
+		)
+		(pin "13"
+		)
+		(pin "60"
+		)
+		(pin "30"
+		)
+		(pin "63"
+		)
+		(pin "65"
+		)
+		(pin "7"
+		)
+		(pin "16"
+		)
+		(pin "31"
+		)
+		(pin "8"
+		)
+		(pin "36"
+		)
+		(pin "9"
+		)
+		(instances
+			(project ""
+				(path "/d34d8324-c983-4098-8d7e-5c2fbd34794d/41f449fb-b4c2-4d53-966f-b49577e16db6"
+					(reference "U4")
+					(unit 1)
+				)
